File: pcb/control_and_power/control_and_power/control_and_power_extended/control_and_power_extended.kicad_pcb (KiCad board)
At the start: 2 copper layers, 51 parts, among them J1 Conn_01x07_Male, Q1 TIP122, Q2 TIP122, Q3 TIP122, Q4 TIP122, Q5 TIP122, Q6 TIP122, U1 4N25, U2 4N25, U3 40106, U4 4N25, U5 4N25, U6 4N25, U7 4N25

Commit message: update, testing pcb components layout and extended control and power pcb
Parts:
- moved U3 83.5 mm to (180.7, 85.9)
- moved D2 80.8 mm to (205.5, 72.4), turned to 180 degrees
- moved R23 76.4 mm to (196.7, 110.4)
- moved D1 74.4 mm to (205.1, 60.0), turned to 180 degrees
- moved R6 73.6 mm to (191.1, 78.2)
- moved J1 73.5 mm to (149.9, 94.6), turned to 0 degrees
- moved R5 69.5 mm to (191.1, 65.7)
- moved 5V1 68.9 mm to (184.2, 62.7), turned to 180 degrees
- moved D5 65.7 mm to (160.1, 50.5)
- moved R24 65.7 mm to (196.4, 122.5)
- moved D6 64.0 mm to (205.6, 122.5), turned to 180 degrees
- moved R8 63.4 mm to (197.0, 72.4)
- moved R20 56.6 mm to (192.0, 128.1)
- moved R19 55.7 mm to (192.0, 115.6)
- moved R16 55.1 mm to (175.0, 106.7)
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Routing:
- net GND: track 0.00 -> 303.5 mm
- net SIG-: track 0.00 -> 116.8 mm
- net 5v: track 0.00 -> 84.3 mm
- net Net-(R9-Pad2): track 0.00 -> 29.4 mm
- net Net-(R10-Pad2): track 0.00 -> 24.6 mm
- net Net-(R11-Pad2): track 0.00 -> 18.4 mm
- net Net-(R2-Pad2): track 0.00 -> 17.8 mm
- net Net-(OUT1-Pad1): track 0.00 -> 12.8 mm
- net Net-(OUT2-Pad1): track 0.00 -> 12.6 mm
- net Net-(R1-Pad2): track 0.00 -> 12.2 mm
- net Net-(OUT3-Pad1): track 0.00 -> 11.6 mm
- net Net-(OUT4-Pad1): track 0.00 -> 11.6 mm
- net Net-(OUT5-Pad1): track 0.00 -> 11.5 mm
- net Net-(OUT6-Pad1): track 0.00 -> 11.4 mm
- net Net-(R12-Pad2): track 0.00 -> 10.1 mm
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
Commit message: backup, updating footprints of extended circuit
Parts:
- added J10: Conn_01x01_Male, Connector_PinHeader_2.54mm:PinHeader_1x01_P2.54mm_Vertical, F.Cu at (201.3, 84.6)
- added J11: Conn_01x01_Male, Connector_PinHeader_2.54mm:PinHeader_1x01_P2.54mm_Vertical, F.Cu at (201.4, 96.9)
- added J12: Conn_01x01_Male, Connector_PinHeader_2.54mm:PinHeader_1x01_P2.54mm_Vertical, F.Cu at (201.3, 121.4)
- added J13: Conn_01x01_Male, Connector_PinHeader_2.54mm:PinHeader_1x01_P2.54mm_Vertical, F.Cu at (201.3, 109.5)
- added J14: Conn_01x01_Male, Connector_PinHeader_2.54mm:PinHeader_1x01_P2.54mm_Vertical, F.Cu at (200.9, 71.2)
- added J15: Conn_01x01_Male, Connector_PinHeader_2.54mm:PinHeader_1x01_P2.54mm_Vertical, F.Cu at (201.3, 57.5)
- added J2: Conn_01x01_Male, Connector_PinHeader_2.54mm:PinHeader_1x01_P2.54mm_Vertical, F.Cu at (176.0, 74.7)
- added J3: Conn_01x01_Male, Connector_PinHeader_2.54mm:PinHeader_1x01_P2.54mm_Vertical, F.Cu at (175.8, 109.6)
- added J4: Conn_01x01_Male, Connector_PinHeader_2.54mm:PinHeader_1x01_P2.54mm_Vertical, F.Cu at (175.8, 118.3)
- added J5: Conn_01x01_Male, Connector_PinHeader_2.54mm:PinHeader_1x01_P2.54mm_Vertical, F.Cu at (175.7, 127.0)
- added J6: Conn_01x01_Male, Connector_PinHeader_2.54mm:PinHeader_1x01_P2.54mm_Vertical, F.Cu at (175.9, 83.5)
- added J7: Conn_01x01_Male, Connector_PinHeader_2.54mm:PinHeader_1x01_P2.54mm_Vertical, F.Cu at (175.9, 91.7)
- added J8: Conn_01x07_Male, Connector_PinHeader_2.54mm:PinHeader_1x07_P2.54mm_Vertical, F.Cu at (183.3, 105.3)
- added J9: Conn_01x07_Male, Connector_PinHeader_2.54mm:PinHeader_1x07_P2.54mm_Vertical, F.Cu at (196.9, 90.0)
- moved D5 88.6 mm to (215.2, 120.0), turned to 180 degrees
- moved R8 21.0 mm to (210.3, 56.0), turned to -90 degrees
- moved R6 20.4 mm to (201.3, 60.5), turned to -90 degrees
- moved R24 20.1 mm to (210.3, 108.1), turned to -90 degrees
- moved D2 19.1 mm to (215.4, 56.0)
- moved OUT6 18.4 mm to (226.1, 65.1)
- moved R20 18.2 mm to (201.2, 112.5), turned to -90 degrees
- moved D6 17.3 mm to (215.1, 108.1)
- moved Q2 16.9 mm to (205.2, 63.0)
- moved OUT4 16.7 mm to (226.0, 116.4)
- moved OUT3 16.6 mm to (226.1, 128.5)
- moved R23 16.6 mm to (210.3, 120.0), turned to -90 degrees
- moved OUT5 16.2 mm to (226.0, 78.9)
- moved R7 15.8 mm to (210.3, 69.7), turned to -90 degrees
- moved D1 14.5 mm to (215.9, 69.7)
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- renumbered OUT3 to OUT1, OUT4 to OUT2, OUT5 to OUT3, OUT6 to OUT4, OUT1 to OUT5, OUT2 to OUT6, U4 to Opto1, U5 to Opto2, U6 to Opto3, U7 to Opto4, U1 to Opto5, U2 to Opto6
Connections:
- net Net-(R13-Pad1) renamed pullup1
- net Net-(R14-Pad1) renamed pullup2
- net Net-(R15-Pad1) renamed pullup3
- net Net-(R16-Pad1) renamed pullup4
- net Net-(R17-Pad1) renamed SOut1
- net Net-(R18-Pad1) renamed SOut2
- net Net-(R19-Pad1) renamed SOut3
- net Net-(R20-Pad1) renamed SOut4
- net Net-(R3-Pad1) renamed pullup5
- net Net-(R4-Pad1) renamed pullup6
- net Net-(R5-Pad1) renamed SOut5
- net Net-(R6-Pad1) renamed SOut6
Routing:
- net 5v: track 84.3 -> 265.8 mm
- net GND: track 303.5 -> 371.1 mm
- net pullup5: track 2.16 -> 27.4 mm, vias 1 -> 0
- net SOut2: track 4.87 -> 21.0 mm, vias 2 -> 0
- net Net-(R2-Pad2): track 17.8 -> 31.1 mm
- net Net-(R1-Pad2): track 12.2 -> 25.3 mm
- net Net-(OUT2-Pad1): track 11.6 -> 21.0 mm
- net Net-(OUT3-Pad1): track 11.5 -> 20.9 mm
- net Net-(OUT1-Pad1): track 11.6 -> 21.0 mm
- net Net-(OUT4-Pad1): track 11.4 -> 20.8 mm
- net Net-(OUT6-Pad1): track 12.6 -> 21.1 mm
- net Net-(OUT5-Pad1): track 12.8 -> 21.2 mm
- net Net-(R12-Pad2): track 10.1 -> 18.0 mm
- net SOut5: track 0.00 -> 5.98 mm
- net Net-(R10-Pad2): track 24.6 -> 18.7 mm
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Other:
- board text added: "O1"
- board text added: "O2"
- board text added: "O3"
- board text added: "O4"
- board text added: "O5"
- board text added: "O6"
- board text added: "OUT1"
- board text added: "OUT2"
- board text added: "OUT3"
- board text added: "OUT4"
- board text added: "OUT5"
- board text added: "OUT6"
- board text added: "S-"
- board text added: "S1"
- board text added: "S2"
- board text added: "S3"
- board text added: "S4"
- board text added: "S5"
- board text added: "S6"
