File: pcb/control_and_power/control_and_power/control_and_power_extended/control_and_power_extended.kicad_sch (KiCad schematic)
At the start: 51 parts, among them J1 Conn_01x07_Male, Q1 TIP122, Q2 TIP122, Q3 TIP122, Q4 TIP122, Q5 TIP122, Q6 TIP122, U1 4N25, U2 4N25, U3 40106, U4 4N25, U5 4N25, U6 4N25, U7 4N25

Commit message: update, testing pcb components layout and extended control and power pcb
Parts:
- J1: footprint (none) -> Connector_PinHeader_2.54mm:PinHeader_1x07_P2.54mm_Vertical
Changed lines of the file:
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@@
     (property "Reference" "J1" (id 0) (at 34.29 38.1 0))
     (property "Value" "Conn_01x07_Male" (id 1) (at 34.29 40.64 0))
-    (property "Footprint" "" (id 2) (at 29.21 53.34 0)
+    (property "Footprint" "Connector_PinHeader_2.54mm:PinHeader_1x07_P2.54mm_Vertical" (id 2) (at 29.21 53.34 0)
       (effects (font (size 1.27 1.27)) hide)
     )

Commit message: backup, updating footprints of extended circuit
Parts:
- added J10, J11, J12, J13, J14, J15, J2, J3, J4, J5, J6, J7: Conn_01x01_Male, Connector_PinHeader_2.54mm:PinHeader_1x01_P2.54mm_Vertical, symbol Connector:Conn_01x01_Male
- added J8, J9: Conn_01x07_Male, Connector_PinHeader_2.54mm:PinHeader_1x07_P2.54mm_Vertical, symbol Connector:Conn_01x07_Male
- renumbered OUT3 to OUT1, OUT4 to OUT2, OUT5 to OUT3, OUT6 to OUT4, OUT1 to OUT5, OUT2 to OUT6, U4 to Opto1, U5 to Opto2, U6 to Opto3, U7 to Opto4, U1 to Opto5, U2 to Opto6
Connections:
- net SOut2: now reaches R18.1, U3.4
- net SOut2: now also J11.1 (Pin_1), J8.4 (Pin_4)
- net pullup3: now reaches Opto3.5, R15.1, U3.5
- net pullup3: now also J7.1 (Pin_1), J8.3 (Pin_3)
- net pullup1: now reaches Opto1.5, R13.1, U3.1
- net pullup1: now also J2.1 (Pin_1), J8.7 (Pin_7)
- net pullup5: now reaches Opto5.5, R3.1, U3.11
- net pullup5: now also J4.1 (Pin_1), J9.4 (Pin_4)
- net SOut3: now reaches R19.1, U3.6
- net SOut3: now also J12.1 (Pin_1), J8.2 (Pin_2)
- net pullup2: now reaches Opto2.5, R14.1, U3.3
- net pullup2: now also J6.1 (Pin_1), J8.5 (Pin_5)
- net pullup6: now reaches Opto6.5, R4.1, U3.13
- net pullup6: now also J5.1 (Pin_1), J9.2 (Pin_2)
- net SOut4: now reaches R20.1, U3.8
- net SOut4: now also J13.1 (Pin_1), J9.7 (Pin_7)
- net pullup4: now reaches Opto4.5, R16.1, U3.9
- net pullup4: now also J3.1 (Pin_1), J9.6 (Pin_6)
- net SOut1: now reaches R17.1, U3.2
- net SOut1: now also J10.1 (Pin_1), J8.6 (Pin_6)
- net SOut5: now reaches R5.1, U3.10
- net SOut5: now also J14.1 (Pin_1), J9.5 (Pin_5)
- net SOut6: now reaches R6.1, U3.12
- net SOut6: now also J15.1 (Pin_1), J9.3 (Pin_3)
Other:
- moved on the sheet: D1, D2, D3, D4, D5, D6, OUT1, OUT2, OUT3, OUT4, OUT5, OUT6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
