File: pcb/2023_s1/lights_control/lights_control/lights_control.kicad_sch (KiCad schematic)
At the start: 9 parts, among them J1 Conn_01x02_Male, Q1 TIP122, U1 4N25, U2 40106

Commit message: addition, added 3 mounting holes to the pcb, need to add voltage reduction and a better transistor to turn on and off the led lights
Parts:
- added H1, H2, H3: MountingHole, MountingHole:MountingHole_2.2mm_M2_Pad, symbol Mechanical:MountingHole
Changed lines of the file:
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@@
     (pin "7")
+  )
+  (symbol (lib_id "Mechanical:MountingHole") (at 62.23 118.11 0) (unit 1)
+    (in_bom yes) (on_board yes) (fields_autoplaced)
+    (property "Reference" "H3" (id 0) (at 64.77 116.8399 0)
+      (effects (font (size 1.27 1.27)) (justify left))
+    )
+    (property "Value" "MountingHole" (id 1) (at 64.77 119.3799 0)
+      (effects (font (size 1.27 1.27)) (justify left))
+    )
+    (property "Footprint" "MountingHole:MountingHole_2.2mm_M2_Pad" (id 2) (at 62.23 118.11 0)
+      (effects (font (size 1.27 1.27)) hide)
+    )
+    (property "Datasheet" "~" (id 3) (at 62.23 118.11 0)
+      (effects (font (size 1.27 1.27)) hide)
+    )
+  )
+  (symbol (lib_id "Mechanical:MountingHole") (at 62.23 111.76 0) (unit 1)
+    (in_bom yes) (on_board yes) (fields_autoplaced)
+    (property "Reference" "H2" (id 0) (at 64.77 110.4899 0)
+      (effects (font (size 1.27 1.27)) (justify left))
+    )
+    (property "Value" "MountingHole" (id 1) (at 64.77 113.0299 0)
+      (effects (font (size 1.27 1.27)) (justify left))
+    )
+    (property "Footprint" "MountingHole:MountingHole_2.2mm_M2_Pad" (id 2) (at 62.23 111.76 0)
+      (effects (font (size 1.27 1.27)) hide)
+    )
+    (property "Datasheet" "~" (id 3) (at 62.23 111.76 0)
+      (effects (font (size 1.27 1.27)) hide)
+    )
   )
   (symbol (lib_id "4xxx:40106") (at 146.05 80.01 0) (unit 1)
@@
     (pin "14")
     (pin "7")
+  )
+  (symbol (lib_id "Mechanical:MountingHole") (at 62.23 105.41 0) (unit 1)
+    (in_bom yes) (on_board yes) (fields_autoplaced)
+    (property "Reference" "H1" (id 0) (at 64.77 104.1399 0)
+      (effects (font (size 1.27 1.27)) (justify left))
+    )
+    (property "Value" "MountingHole" (id 1) (at 64.77 106.6799 0)
+      (effects (font (size 1.27 1.27)) (justify left))
+    )
+    (property "Footprint" "MountingHole:MountingHole_2.2mm_M2_Pad" (id 2) (at 62.23 105.41 0)
+      (effects (font (size 1.27 1.27)) hide)
+    )
+    (property "Datasheet" "~" (id 3) (at 62.23 105.41 0)
+      (effects (font (size 1.27 1.27)) hide)
+    )
   )
   (symbol (lib_id "Connector:Conn_01x02_Male") (at 64.77 83.82 180) (unit 1)
@@
       (reference "12V1") (unit 1) (value "Screw_Terminal_01x02") (footprint "TerminalBlock:TerminalBlock_Altech_AK300-2_P5.00mm")
     )
+    (path "/be49ff53-de06-4606-ab2e-9292d996c64b"
+      (reference "H1") (unit 1) (value "MountingHole") (footprint "MountingHole:MountingHole_2.2mm_M2_Pad")
+    )
+    (path "/4cd79eee-8923-4e09-a2a6-cd02df77fc65"
+      (reference "H2") (unit 1) (value "MountingHole") (footprint "MountingHole:MountingHole_2.2mm_M2_Pad")
+    )
+    (path "/374cf5fa-e379-4130-89db-81c0afcf3b77"
+      (reference "H3") (unit 1) (value "MountingHole") (footprint "MountingHole:MountingHole_2.2mm_M2_Pad")
+    )
     (path "/c0d85d48-f487-4977-b7ac-02dde425706b"

Commit message: update, new export files and added voltage elevator space for lights control pcb
Parts:
- added H? (x4): MountingHole, MountingHole:MountingHole_2.2mm_M2_Pad, symbol Mechanical:MountingHole
Changed lines of the file:
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@@
+    )
+  )
+  (symbol (lib_id "Mechanical:MountingHole") (at 51.816 145.288 0) (unit 1)
+    (in_bom yes) (on_board yes) (fields_autoplaced)
+    (property "Reference" "H?" (id 0) (at 54.356 144.0179 0)
+      (effects (font (size 1.27 1.27)) (justify left))
+    )
+    (property "Value" "MountingHole" (id 1) (at 54.356 146.5579 0)
+      (effects (font (size 1.27 1.27)) (justify left))
+    )
+    (property "Footprint" "MountingHole:MountingHole_2.2mm_M2_Pad" (id 2) (at 51.816 145.288 0)
+      (effects (font (size 1.27 1.27)) hide)
+    )
+    (property "Datasheet" "~" (id 3) (at 51.816 145.288 0)
+      (effects (font (size 1.27 1.27)) hide)
     )
   )
@@
     (pin "7")
   )
+  (symbol (lib_id "Mechanical:MountingHole") (at 51.816 139.7 0) (unit 1)
+    (in_bom yes) (on_board yes) (fields_autoplaced)
+    (property "Reference" "H?" (id 0) (at 54.356 138.4299 0)
+      (effects (font (size 1.27 1.27)) (justify left))
+    )
+    (property "Value" "MountingHole" (id 1) (at 54.356 140.9699 0)
+      (effects (font (size 1.27 1.27)) (justify left))
+    )
+    (property "Footprint" "MountingHole:MountingHole_2.2mm_M2_Pad" (id 2) (at 51.816 139.7 0)
+      (effects (font (size 1.27 1.27)) hide)
+    )
+    (property "Datasheet" "~" (id 3) (at 51.816 139.7 0)
+      (effects (font (size 1.27 1.27)) hide)
+    )
+  )
   (symbol (lib_id "Connector:Screw_Terminal_01x02") (at 57.15 64.77 180) (unit 1)
     (in_bom yes) (on_board yes)
@@
     (pin "2")
   )
+  (symbol (lib_id "Mechanical:MountingHole") (at 51.816 149.86 0) (unit 1)
+    (in_bom yes) (on_board yes) (fields_autoplaced)
+    (property "Reference" "H?" (id 0) (at 54.356 148.5899 0)
+      (effects (font (size 1.27 1.27)) (justify left))
+    )
+    (property "Value" "MountingHole" (id 1) (at 54.356 151.1299 0)
+      (effects (font (size 1.27 1.27)) (justify left))
+    )
+    (property "Footprint" "MountingHole:MountingHole_2.2mm_M2_Pad" (id 2) (at 51.816 149.86 0)
+      (effects (font (size 1.27 1.27)) hide)
+    )
+    (property "Datasheet" "~" (id 3) (at 51.816 149.86 0)
+      (effects (font (size 1.27 1.27)) hide)
+    )
+  )
   (symbol (lib_id "4xxx:40106") (at 149.86 113.03 0) (unit 5)
     (in_bom yes) (on_board yes) (fields_autoplaced)
@@
     (pin "14")
     (pin "7")
+  )
+  (symbol (lib_id "Mechanical:MountingHole") (at 51.816 134.366 0) (unit 1)
+    (in_bom yes) (on_board yes) (fields_autoplaced)
+    (property "Reference" "H?" (id 0) (at 54.356 133.0959 0)
+      (effects (font (size 1.27 1.27)) (justify left))
+    )
+    (property "Value" "MountingHole" (id 1) (at 54.356 135.6359 0)
+      (effects (font (size 1.27 1.27)) (justify left))
+    )
+    (property "Footprint" "MountingHole:MountingHole_2.2mm_M2_Pad" (id 2) (at 51.816 134.366 0)
+      (effects (font (size 1.27 1.27)) hide)
+    )
+    (property "Datasheet" "~" (id 3) (at 51.816 134.366 0)
+      (effects (font (size 1.27 1.27)) hide)
+    )
   )
   (symbol (lib_id "Mechanical:MountingHole") (at 62.23 105.41 0) (unit 1)
@@
       (reference "H3") (unit 1) (value "MountingHole") (footprint "MountingHole:MountingHole_2.2mm_M2_Pad")
     )
+    (path "/0f2fcff6-4797-4938-b61d-80cbd1d8e037"
+      (reference "H?") (unit 1) (value "MountingHole") (footprint "MountingHole:MountingHole_2.2mm_M2_Pad")
+    )
+    (path "/5dac930c-c4d0-4e22-bc0d-75285312ea29"
+      (reference "H?") (unit 1) (value "MountingHole") (footprint "MountingHole:MountingHole_2.2mm_M2_Pad")
+    )
+    (path "/8cd22167-a260-4c55-b1df-8df68a85fa7f"
+      (reference "H?") (unit 1) (value "MountingHole") (footprint "MountingHole:MountingHole_2.2mm_M2_Pad")
+    )
+    (path "/93dcfb43-2ed0-43c5-b01a-56e8eb3c160b"
+      (reference "H?") (unit 1) (value "MountingHole") (footprint "MountingHole:MountingHole_2.2mm_M2_Pad")
+    )
     (path "/c0d85d48-f487-4977-b7ac-02dde425706b"

Commit message: update, routed lights pcb
Parts:
- removed J1: Conn_01x02_Male, Connector_JST:JST_EH_B2B-EH-A_1x02_P2.50mm_Vertical, symbol Connector:Conn_01x02_Male
- added 12V2, 12V3: Screw_Terminal_01x02, TerminalBlock_Altech:Altech_AK300_1x02_P5.00mm_45-Degree, symbol Connector:Screw_Terminal_01x02
- 12V1, OUT1: footprint TerminalBlock:TerminalBlock_Altech_AK300-2_P5.00mm -> TerminalBlock_Altech:Altech_AK300_1x02_P5.00mm_45-Degree
- gave numbers to parts that had none: 4
Connections:
- net 5v: now also 12V3.1 (Pin_1)
- net D26: now also 12V2.2 (Pin_2)
- net GND5V: now also 12V2.1 (Pin_1), 12V3.2 (Pin_2)
Other:
- moved on the sheet: 12V1, H1, H2, H3, H4, H5, H6, H7, U2B, U2C, U2D, U2E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

Commit message: update, fixed lights pcb, only lacks rerouting
Parts:
- removed 12V3: Screw_Terminal_01x02, TerminalBlock_Altech:Altech_AK300_1x02_P5.00mm_45-Degree, symbol Connector:Screw_Terminal_01x02
Connections:
- net 5v is gone; now on net 12v: R2.2, U2.14 (VDD)
- net GND12V: now also U1.4, U2.7 (VSS)
- net GND5V renamed GND SIG
- net GND SIG: no longer U1.4, U2.7 (VSS)
Other:
- moved on the sheet: 12V1, 12V2, H1, H2, H3, H4, H5, H6, H7, U2B, U2C, U2D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
