File: pcb/control_and_power/control_and_power/control_and_power.kicad_sch (KiCad schematic)
At the start: 12 parts, among them Q1 TIP122, U1 40106, U2 4N25

Commit message: update, fixed lights pcb, only lacks rerouting
Other:
- moved on the sheet: U1B, U1C, U1D, U1E, U1F, U1G
