File: pcb/2023/integration/integration_with_esp32_only/intregration1.kicad_pcb (KiCad board)
At the start: 2 copper layers, 41 parts, among them J1 Screw_Terminal_01x03, J2 Screw_Terminal_01x03, J4 Screw_Terminal_01x02, Q1 2N2219, Q2 2N2219, Q3 2N2219, Q4 2N2219

Commit message: update, rerouted paths and added text to the pcb
Parts:
- 5V1, C1, C2, D1, D2, D3, D4, H1, H2, H3, H4, H5, H6, J1, J2, J4, J_AC_INPUT1, J_LOAD1, J_LOAD2, J_esp0, J_esp1, J_fan1, J_oxygen1, J_wpump1, K_LIGHTS1, Q1, Q2, Q3, Q4, R1, R2, R3, R4, R5, R6, R7, R8, R9, U_fan1, U_oxygen1, U_wpump1: moved to F.Cu
- moved R6 105.4 mm to (156.2, 130.3)
- moved H2 99.5 mm to (54.0, 31.6), turned to 0 degrees
- moved H5 99.0 mm to (54.1, 96.3), turned to 0 degrees
- moved H1 98.9 mm to (153.1, 31.6), turned to 0 degrees
- moved H6 98.4 mm to (152.8, 96.0), turned to 0 degrees
- moved J_LOAD1 94.6 mm to (56.2, 161.3), turned to 0 degrees
- moved U_fan1 91.5 mm to (149.3, 136.7)
- moved Q1 90.2 mm to (148.6, 106.7)
- moved K_LIGHTS1 83.3 mm to (61.9, 130.3)
- moved J_fan1 82.2 mm to (144.6, 161.3), turned to 0 degrees
- moved D1 81.3 mm to (144.1, 130.0)
- moved R2 72.5 mm to (139.8, 104.3)
- moved H3 70.4 mm to (138.7, 147.3), turned to 0 degrees
- moved J_LOAD2 64.3 mm to (71.3, 161.3), turned to 0 degrees
- moved R8 64.3 mm to (135.6, 130.3)
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Routing:
- net GND5V: track 238.4 -> 313.1 mm, vias 0 -> 2
- net 5v: track 314.0 -> 370.4 mm, vias 9 -> 7
- net D23: track 24.5 -> 72.9 mm, vias 0 -> 2
- net D34: track 68.1 -> 42.5 mm
- net D25: track 68.3 -> 44.4 mm
- net D18: track 53.8 -> 51.3 mm
- net Net-(J_fan1-Pin_2): track 11.6 -> 14.0 mm
- net AC1: track 71.6 -> 73.7 mm
- net Net-(J_wpump1-Pin_2): track 11.6 -> 13.6 mm
- net Net-(J_oxygen1-Pin_2): track 11.7 -> 13.7 mm
- net Normally O: track 30.2 -> 31.4 mm
- net AC2: track 65.5 -> 64.6 mm
- net LOAD IN: track 38.5 -> 39.1 mm
Other:
- board text added: "23"
- board text added: "25"
- board text added: "34"
- board text added: "5V"
- board text added: "AC OUT"
- board text added: "AC-IN"
- board text added: "GND"
- board text added: "LOAD-IN"
- board text added: "LOAD-OUT"

Commit message: add, added second revision integration pcb update
Parts:
- removed C1: C_Polarized, Capacitor_THT:CP_Radial_D5.0mm_P2.50mm
- removed C2: C_Generic, Capacitor_THT:C_Disc_D5.0mm_W2.5mm_P2.50mm
- removed R6, R7, R8: R, Resistor_THT:R_Axial_DIN0204_L3.6mm_D1.6mm_P5.08mm_Vertical
- added D6: 1N53xxB, Diode_THT:D_DO-201_P15.24mm_Horizontal, B.Cu at (126.4, 37.5)
- 5V1, D1, D2, D3, D4, H1, H2, H3, H4, H5, H6, J1, J2, J4, J_AC_INPUT1, J_LOAD1, J_LOAD2, J_esp0, J_esp1, J_fan1, J_oxygen1, J_wpump1, Q1, Q2, Q3, Q4, R1, R2, R3, R4, R5: moved to B.Cu
- K_LIGHTS1: value SANYOU_SRD_Form_C -> JQC-3F; moved to B.Cu
- R9: value R -> 20; moved to B.Cu
- U_fan1, U_oxygen1, U_wpump1: value 34.81-8240 -> G3MB-202P; moved to B.Cu
- moved H1 99.3 mm to (53.9, 31.6), turned to 180 degrees
- moved H2 99.1 mm to (153.0, 31.6), turned to 180 degrees
- moved H5 98.9 mm to (152.9, 96.3), turned to 180 degrees
- moved H6 98.5 mm to (54.2, 96.0), turned to 180 degrees
- moved J_LOAD1 94.6 mm to (150.8, 161.3), turned to 180 degrees
- moved U_fan1 91.5 mm to (57.7, 136.7)
- moved Q1 90.2 mm to (58.4, 106.7)
- moved J4 86.4 mm to (146.7, 50.7)
- moved J1 86.1 mm to (146.6, 77.1)
- moved J2 86.1 mm to (146.6, 59.3)
- moved K_LIGHTS1 83.3 mm to (145.1, 130.3)
- moved J_fan1 82.2 mm to (62.4, 161.3), turned to 180 degrees
- moved D1 81.3 mm to (62.9, 130.0)
- moved R2 72.5 mm to (67.2, 104.3)
- moved H3 70.4 mm to (68.3, 147.3), turned to 180 degrees
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Connections:
- D1 pad 1: Net-(D1-K) -> 5v
- D2 pad 1: Net-(D2-K) -> 5v
- D3 pad 1: Net-(D3-K) -> 5v
- U_fan1 pad A1: Net-(D1-K) -> 5v
- U_oxygen1 pad A1: Net-(D3-K) -> 5v
- U_wpump1 pad A1: Net-(D2-K) -> 5v
Routing:
- net GND5V: track 313.1 -> 268.3 mm, vias 2 -> 3
- net 5v: track 370.4 -> 338.8 mm, vias 7 -> 2
- net Net-(D2-K): track 13.6 -> 0.00 mm
- net Net-(D3-K): track 12.7 -> 0.00 mm
- net Net-(D1-K): track 12.1 -> 0.00 mm
