File: pcb/2023/integration/integration_with_esp32_only/intregration1.kicad_sch (KiCad schematic)
At the start: 41 parts, among them J1 Screw_Terminal_01x02, Q1 2N2219, Q2 2N2219, Q3 2N2219, Q4 2N2219

Commit message: update, rerouted paths and added text to the pcb
Other:
- moved on the sheet: D1, D2, D3, J?, J_fan1, J_oxygen1, J_wpump1, Q1, Q3, Q4, R1, R11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

Commit message: add, added second revision integration pcb update
Parts:
- removed C1: C_Polarized, Capacitor_THT:CP_Radial_D5.0mm_P2.50mm, symbol Device:C_Polarized
- removed C2: C_Generic, Capacitor_THT:C_Disc_D5.0mm_W2.5mm_P2.50mm, symbol PCM_4ms_Capacitor:C_Generic
- removed R5, R7, R9: R, Resistor_THT:R_Axial_DIN0204_L3.6mm_D1.6mm_P5.08mm_Vertical, symbol Device:R
- added D6: 1N53xxB, Diode_THT:D_DO-201_P15.24mm_Horizontal, symbol Diode:1N53xxB
- K_LIGHTS1: value SANYOU_SRD_Form_C -> JQC-3F
- R6: value R -> 20
- U_fan1, U_oxygen1, U_wpump1: value 34.81-8240 -> G3MB-202P
Connections:
- net 5v: now also D1.1 (K), D2.1 (K), D3.1 (K), U_fan1.A1, U_oxygen1.A1, U_wpump1.A1, D6.1 (K)
- net GND5V: now also D6.2 (A)
Other:
- moved on the sheet: 5V1, D1, D2, D3, D4, H1, H2, H3, H4, J1, J_AC_INPUT1, J_LOAD1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
